File: projects/jlcpcb/jlcpcb.kicad_pcb (KiCad board)
At the start: 2 copper layers, 0 parts

Commit message: Added IPS 240x240 Display Part and Footprint
Other:
- net class Default: trace_width 0.127 -> 0.1524
Changed lines of the file:
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@@
-(kicad_pcb (version 20171130) (host pcbnew "(5.1.6-0-10_14)")
+(kicad_pcb (version 20171130) (host pcbnew "(5.1.9)-1")
   (general
     (thickness 1.6)
@@
   )
   (setup
-    (last_trace_width 0.127)
+    (last_trace_width 0.1524)
+    (user_trace_width 0.127)
     (user_trace_width 0.3048)
+    (user_trace_width 0.381)
     (trace_clearance 0.127)
     (zone_clearance 0.508)
@@
     (pad_to_mask_clearance 0.05)
     (aux_axis_origin 0 0)
-    (visible_elements FFFFFF7F)
+    (visible_elements 7FFFFFFF)
     (pcbplotparams
       (layerselection 0x010fc_ffffffff)
@@
   (net_class Default "This is the default net class."
     (clearance 0.127)
-    (trace_width 0.127)
+    (trace_width 0.1524)
     (via_dia 0.6096)
     (via_drill 0.3048)

Commit message: changed preset values
Other:
- net class Default: via_dia 0.6096 -> 0.6; via_drill 0.3048 -> 0.3
- net class Power: via_dia 0.762 -> 0.6; via_drill 0.381 -> 0.3
- rule via_min_drill: 0.3048 -> 0.3
- rule via_min_size: 0.6096 -> 0.6
Changed lines of the file:
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@@
-(kicad_pcb (version 20171130) (host pcbnew "(5.1.9)-1")
+(kicad_pcb (version 20171130) (host pcbnew "(5.1.6-0-10_14)")
   (general
     (thickness 1.6)
@@
     (last_trace_width 0.1524)
     (user_trace_width 0.127)
+    (user_trace_width 0.1524)
     (user_trace_width 0.3048)
     (user_trace_width 0.381)
@@
     (zone_45_only no)
     (trace_min 0.127)
-    (via_size 0.6096)
-    (via_drill 0.3048)
-    (via_min_size 0.6096)
-    (via_min_drill 0.3048)
+    (via_size 0.6)
+    (via_drill 0.3)
+    (via_min_size 0.6)
+    (via_min_drill 0.3)
+    (user_via 0.6 0.3)
     (user_via 0.762 0.381)
-    (uvia_size 0.6096)
-    (uvia_drill 0.3048)
+    (uvia_size 0.6)
+    (uvia_drill 0.3)
     (uvias_allowed no)
     (uvia_min_size 0.2)
@@
     (clearance 0.127)
     (trace_width 0.1524)
-    (via_dia 0.6096)
-    (via_drill 0.3048)
-    (uvia_dia 0.6096)
-    (uvia_drill 0.3048)
-    (diff_pair_width 0.127)
+    (via_dia 0.6)
+    (via_drill 0.3)
+    (uvia_dia 0.6)
+    (uvia_drill 0.3)
+    (diff_pair_width 0.1524)
     (diff_pair_gap 0.127)
   )
@@
     (clearance 0.254)
     (trace_width 0.3048)
-    (via_dia 0.762)
-    (via_drill 0.381)
-    (uvia_dia 0.762)
-    (uvia_drill 0.381)
+    (via_dia 0.6)
+    (via_drill 0.3)
+    (uvia_dia 0.6)
+    (uvia_drill 0.3)
     (diff_pair_width 0.3048)
     (diff_pair_gap 0.254)
