File: projects/jlcpcb/jlcpcb.kicad_pcb (KiCad board)
At the start: 2 copper layers, 0 parts

Commit message: new stuff
Other:
- rule via_min_drill: 0.3 -> 0.2
- rule via_min_size: 0.6 -> 0.4
Changed lines of the file:
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@@
-(kicad_pcb (version 20171130) (host pcbnew "(5.1.6-0-10_14)")
+(kicad_pcb (version 20171130) (host pcbnew "(5.1.9-0-10_14)")
   (general
     (thickness 1.6)
@@
     (via_size 0.6)
     (via_drill 0.3)
-    (via_min_size 0.6)
-    (via_min_drill 0.3)
+    (via_min_size 0.4)
+    (via_min_drill 0.2)
+    (user_via 0.4 0.2)
     (user_via 0.6 0.3)
     (user_via 0.762 0.381)
@@
     (uvia_drill 0.3)
     (uvias_allowed no)
-    (uvia_min_size 0.6)
-    (uvia_min_drill 0.3)
+    (uvia_min_size 0.4)
+    (uvia_min_drill 0.2)
     (edge_width 0.05)
     (segment_width 0.2)
