File: projects/jlcpcb4layer/jlcpcb4layer.kicad_pcb (KiCad board)
At the start: 2 copper layers, 0 parts

Commit message: added 4 layer jlcpcb template
Other:
- copper layers 2 -> 4
- net class Minimal added: clearance 0.127, trace_width 0.127, via_dia 0.45, via_drill 0.2
- rule via_min_drill: 0.3 -> 0.2
- rule via_min_size: 0.6 -> 0.45
Changed lines of the file:
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@@
   (layers
     (0 F.Cu signal)
+    (1 In1.Cu signal)
+    (2 In2.Cu signal)
     (31 B.Cu signal)
     (32 B.Adhes user)
@@
     (via_size 0.6)
     (via_drill 0.3)
-    (via_min_size 0.6)
-    (via_min_drill 0.3)
+    (via_min_size 0.45)
+    (via_min_drill 0.2)
+    (user_via 0.45 0.2)
     (user_via 0.6 0.3)
     (user_via 0.762 0.381)
@@
     (uvia_drill 0.3)
     (uvias_allowed no)
-    (uvia_min_size 0.6)
-    (uvia_min_drill 0.3)
+    (uvia_min_size 0.45)
+    (uvia_min_drill 0.2)
     (edge_width 0.05)
     (segment_width 0.2)
@@
     (pad_to_mask_clearance 0.05)
     (aux_axis_origin 0 0)
-    (visible_elements 7FFFFFFF)
+    (visible_elements FFFFFF7F)
     (pcbplotparams
       (layerselection 0x010fc_ffffffff)
@@
     (diff_pair_gap 0.127)
   )
+  (net_class Minimal ""
+    (clearance 0.127)
+    (trace_width 0.127)
+    (via_dia 0.45)
+    (via_drill 0.2)
+    (uvia_dia 0.45)
+    (uvia_drill 0.2)
+    (diff_pair_width 0.127)
+    (diff_pair_gap 0.127)
+  )
